Commit message: Correct Z1 joint limits

File: rtb-data/rtbdata/xacro/z1_description/xacro/const.xacro (robot description, xacro)
@@ -113,10 +113,10 @@
     <xacro:property name="joint2_PositionMin" value="0.0"/>
     <xacro:property name="joint2_PositionMax" value="${PI}"/>
-    <xacro:property name="joint3_PositionMin" value="${-PI*274/180}"/>
+    <xacro:property name="joint3_PositionMin" value="${-PI*165/180}"/>
     <xacro:property name="joint3_PositionMax" value="0.0"/>
-    <xacro:property name="joint4_PositionMin" value="${-PI*100/180}"/>
-    <xacro:property name="joint4_PositionMax" value="${PI*90/180}"/>
-    <xacro:property name="joint5_PositionMin" value="${-PI*99/180}"/>
-    <xacro:property name="joint5_PositionMax" value="${PI*99/180}"/>
+    <xacro:property name="joint4_PositionMin" value="${-PI*87/180}"/>
+    <xacro:property name="joint4_PositionMax" value="${PI*87/180}"/>
+    <xacro:property name="joint5_PositionMin" value="${-PI*77/180}"/>
+    <xacro:property name="joint5_PositionMax" value="${PI*77/180}"/>
     <xacro:property name="joint6_PositionMin" value="${-PI*160/180}"/>
     <xacro:property name="joint6_PositionMax" value="${PI*160/180}"/>
